Commit message: v1.0.1: pin robot descriptions in the workspace, re-render m5 clips
- src/external/{robotiq_description,ur_description}: git submodules at the jazzy release tags
  (release/jazzy/robotiq_description/0.0.1-3, release/jazzy/ur_description/3.5.1-1). The overlay takes
  precedence over the system (Isaac) builds; no apt changes needed. ros2 pkg prefix -> install/.
- gen_gripper_urdf.py: store package:// mesh URIs (robotiq 0.0.1 writes absolute file:// paths); regenerated
  gripper xacro differs only in the 9 visual mesh paths; expanded URDF otherwise identical (FK unchanged).
- New test: every URDF mesh resolves into the workspace, never /opt/ros. Clean rebuild: 60/60 tests pass.
- m5 clips re-rendered with the wrist-camera bracket; commands in docs/m5_catch.md.
- README prerequisites + docs/m0_toolchain.md: no special apt versions, descriptions pinned in src/external.

File: src/catch_description/urdf/robotiq_2f85_catch.xacro (robot description, xacro)
@@ -7,5 +7,5 @@
     <visual>
       <geometry>
-        <mesh filename="package://robotiq_description/meshes/visual/2f_85/robotiq_base.dae" />
+        <mesh filename="package://robotiq_description/meshes/visual/robotiq_base.dae" />
       </geometry>
     </visual>
@@ -19,5 +19,5 @@
     <visual>
       <geometry>
-        <mesh filename="package://robotiq_description/meshes/visual/2f_85/left_knuckle.dae" />
+        <mesh filename="package://robotiq_description/meshes/visual/left_knuckle.dae" />
       </geometry>
     </visual>
@@ -31,5 +31,5 @@
     <visual>
       <geometry>
-        <mesh filename="package://robotiq_description/meshes/visual/2f_85/right_knuckle.dae" />
+        <mesh filename="package://robotiq_description/meshes/visual/right_knuckle.dae" />
       </geometry>
     </visual>
@@ -43,5 +43,5 @@
     <visual>
       <geometry>
-        <mesh filename="package://robotiq_description/meshes/visual/2f_85/left_finger.dae" />
+        <mesh filename="package://robotiq_description/meshes/visual/left_finger.dae" />
       </geometry>
     </visual>
@@ -55,5 +55,5 @@
     <visual>
       <geometry>
-        <mesh filename="package://robotiq_description/meshes/visual/2f_85/right_finger.dae" />
+        <mesh filename="package://robotiq_description/meshes/visual/right_finger.dae" />
       </geometry>
     </visual>
@@ -67,5 +67,5 @@
     <visual>
       <geometry>
-        <mesh filename="package://robotiq_description/meshes/visual/2f_85/left_inner_knuckle.dae" />
+        <mesh filename="package://robotiq_description/meshes/visual/left_inner_knuckle.dae" />
       </geometry>
     </visual>
@@ -79,5 +79,5 @@
     <visual>
       <geometry>
-        <mesh filename="package://robotiq_description/meshes/visual/2f_85/right_inner_knuckle.dae" />
+        <mesh filename="package://robotiq_description/meshes/visual/right_inner_knuckle.dae" />
       </geometry>
     </visual>
@@ -91,5 +91,5 @@
     <visual>
       <geometry>
-        <mesh filename="package://robotiq_description/meshes/visual/2f_85/left_finger_tip.dae" />
+        <mesh filename="package://robotiq_description/meshes/visual/left_finger_tip.dae" />
       </geometry>
     </visual>
@@ -103,5 +103,5 @@
     <visual>
       <geometry>
-        <mesh filename="package://robotiq_description/meshes/visual/2f_85/right_finger_tip.dae" />
+        <mesh filename="package://robotiq_description/meshes/visual/right_finger_tip.dae" />
       </geometry>
     </visual>
