Commit message: M3: perception (1.7 mm), colour check at B, pick/place skills (6/6), pallets moved, URDF pallet borders

File: src/catch_description/urdf/scene.urdf.xacro (robot description, xacro)
@@ -29,11 +29,37 @@
     size="${scene['table']['size'][0]} ${scene['table']['size'][1]} ${scene['table']['top_thickness']}"
     xyz="0 0 ${top_z - scene['table']['top_thickness'] / 2}"/>
-  <!-- pallets: base plate + one collision box per slot border ring (simplified as the outer plate height) -->
+  <!-- pallets: base plate + 4 border bars per slot (same boxes as the MJCF), all in one link per pallet -->
+  <xacro:macro name="pbox" params="size xyz rgba">
+    <visual><origin xyz="${xyz}"/><geometry><box size="${size}"/></geometry><material name="pb_${rgba}"><color rgba="${rgba}"/></material></visual>
+    <collision><origin xyz="${xyz}"/><geometry><box size="${size}"/></geometry></collision>
+  </xacro:macro>
+  <xacro:macro name="slot" params="key idx colors">
+    <xacro:if value="${idx &lt; len(colors)}">
+      <xacro:property name="pl" value="${scene['pallets']}"/>
+      <xacro:property name="cx" value="${(idx - 1) * pl['slot_pitch']}"/>
+      <xacro:property name="bw" value="${pl['border_width']}"/>
+      <xacro:property name="bh" value="${pl['border_height']}"/>
+      <xacro:property name="inner" value="${pl['slot_inner']}"/>
+      <xacro:property name="bz" value="${pl['base_size'][2] + bh / 2}"/>
+      <xacro:property name="half" value="${inner / 2 + bw / 2}"/>
+      <xacro:property name="rgba" value="${' '.join(str(v) for v in scene['cube']['colors'][colors[idx]])}"/>
+      <xacro:pbox size="${inner + 2 * bw} ${bw} ${bh}" xyz="${cx} ${half} ${bz}" rgba="${rgba}"/>
+      <xacro:pbox size="${inner + 2 * bw} ${bw} ${bh}" xyz="${cx} ${-half} ${bz}" rgba="${rgba}"/>
+      <xacro:pbox size="${bw} ${inner} ${bh}" xyz="${cx + half} 0 ${bz}" rgba="${rgba}"/>
+      <xacro:pbox size="${bw} ${inner} ${bh}" xyz="${cx - half} 0 ${bz}" rgba="${rgba}"/>
+      <xacro:slot key="${key}" idx="${idx + 1}" colors="${colors}"/>
+    </xacro:if>
+  </xacro:macro>
   <xacro:macro name="pallet" params="key">
     <xacro:property name="pl" value="${scene['pallets']}"/>
     <xacro:property name="c" value="${pl[key]['center']}"/>
-    <xacro:box_link name="pallet_${key}" rgba="0.8 0.8 0.78 1"
-      size="${pl['base_size'][0]} ${pl['base_size'][1]} ${pl['base_size'][2] + pl['border_height']}"
-      xyz="${c[0]} ${c[1]} ${top_z + (pl['base_size'][2] + pl['border_height']) / 2}"/>
+    <link name="pallet_${key}">
+      <xacro:pbox size="${pl['base_size'][0]} ${pl['base_size'][1]} ${pl['base_size'][2]}"
+        xyz="0 0 ${pl['base_size'][2] / 2}" rgba="0.8 0.8 0.78 1"/>
+      <xacro:slot key="${key}" idx="0" colors="${pl['slot_order']}"/>
+    </link>
+    <joint name="world_to_pallet_${key}" type="fixed">
+      <parent link="world"/><child link="pallet_${key}"/><origin xyz="${c[0]} ${c[1]} ${top_z}"/>
+    </joint>
   </xacro:macro>
   <xacro:pallet key="a"/>

Commit message: M5 (part): catch eval, controller-timed grip loosen (gripper A on a JTC), wrist-camera in-hand pose + corrected place, URDF wrist camera frame, static-only TF in perception, no-weld test

File: src/catch_description/urdf/scene.urdf.xacro (robot description, xacro)
@@ -106,4 +106,24 @@
   <!-- B's wrist camera frame (optical convention: z forward, x right, y down) for perception -->
   <xacro:property name="wc" value="${scene['cameras']['b_wrist']['pos_in_gripper_base']}"/>
+  <!-- The MJCF camera sits at wc in the Menagerie base frame (wc[0] = 0) and looks at the TCP; the TCP frame is
+       that base frame rotated +90 deg about z. Elevation phi of the camera above the TCP, seen from the TCP. -->
+  <xacro:property name="wc_dz" value="${wc[2] - ins['top_z'] - edge / 2}"/>
+  <xacro:property name="wc_phi" value="${atan2(wc_dz, wc[1])}"/>
+  <link name="b_wrist_cam_optical"/>
+  <joint name="b_wrist_cam_optical_joint" type="fixed">
+    <parent link="b_tcp"/><child link="b_wrist_cam_optical"/>
+    <origin xyz="${wc[1]} ${-wc[0]} ${wc_dz}" rpy="${atan2(-cos(wc_phi), -sin(wc_phi))} 0 ${pi / 2}"/>
+  </joint>
+  <!-- camera housing (MJCF: visual only); a collision box here keeps MoveIt conservative around it -->
+  <link name="b_wrist_cam_housing">
+    <visual><geometry><box size="0.024 0.030 0.024"/></geometry>
+      <material name="b_wrist_cam_mat"><color rgba="0.1 0.1 0.1 1"/></material></visual>
+    <collision><geometry><box size="0.030 0.036 0.030"/></geometry></collision>
+  </link>
+  <joint name="b_wrist_cam_housing_joint" type="fixed">
+    <parent link="b_wrist_cam_optical"/><child link="b_wrist_cam_housing"/>
+    <!-- MJCF housing: 14 mm behind the lens along the view axis, box axes = Menagerie base axes -->
+    <origin xyz="0 0 -0.014" rpy="${-atan2(-cos(wc_phi), -sin(wc_phi))} 0 0"/>
+  </joint>
   <xacro:if value="$(arg ros2_control)">
     <ros2_control name="MujocoSystem" type="system">

Commit message: M5: contact-triggered cup catch 30/30, wrist-camera in-hand pose, corrected place 30/30 in slot (yaw 0.00 deg)
- Catch: B pre-positions from the throw-plan preview (elbow-up cup pose), closes on the palm force sensor
  (2 s queue, subscribed per goal); no weld (tested). 30 throws, 10 per color: 30/30 caught, trigger
  -2.7 +- 0.7 ms vs predicted arrival; time-trigger baseline 30/30 but its close instant scatters up to +50 ms.
- In-hand pose from B's wrist camera (square fit on the face plane, reliable edges only, physical gate):
  angle error <= 0.75 deg / 0.3 mm (<= 0.7 deg up to 18 deg in the hand). Corrected place 30/30 in slot,
  x -0.70 +- 0.07 mm, yaw 0.00 deg; off-centre catches corrected 9/9 vs uncorrected 0/9 in slot.
- Grip loosen of the throw scheduled by the controller (gripper A on a JTC): a Python sim-clock sleep was up to
  97 ms late and caused a miss. URDF wrist-camera frame (FK test), /tf_static-only perception TF, B places
  with the closing axis along world y, carry via home, FastDDS SHM cleanup in sim_ctl.
- Tools: catch_eval, recorder + bag_to_npz, replay renderer, catch envelope study, plot_catch, run_m5.sh.

File: src/catch_description/urdf/scene.urdf.xacro (robot description, xacro)
@@ -115,9 +115,9 @@
     <origin xyz="${wc[1]} ${-wc[0]} ${wc_dz}" rpy="${atan2(-cos(wc_phi), -sin(wc_phi))} 0 ${pi / 2}"/>
   </joint>
-  <!-- camera housing (MJCF: visual only); a collision box here keeps MoveIt conservative around it -->
+  <!-- camera housing (MJCF: visual only, 24 x 30 x 24 mm); collision box 1 mm larger per side for MoveIt -->
   <link name="b_wrist_cam_housing">
     <visual><geometry><box size="0.024 0.030 0.024"/></geometry>
       <material name="b_wrist_cam_mat"><color rgba="0.1 0.1 0.1 1"/></material></visual>
-    <collision><geometry><box size="0.030 0.036 0.030"/></geometry></collision>
+    <collision><geometry><box size="0.026 0.032 0.026"/></geometry></collision>
   </link>
   <joint name="b_wrist_cam_housing_joint" type="fixed">

Commit message: v1.0 housekeeping: wrist-camera bracket, top-to-bottom architecture SVG, /clock off the multi-threaded executors
- The object floating near B's gripper in the demo is the wrist-camera housing (b_robotiq_wrist_cam_housing on
  b_robotiq_base). Added an L-bracket holding it to the gripper base: MJCF visual-only boxes (dynamics unchanged),
  URDF visual + collision, SRDF regenerated, URDF/MJCF agreement test for housing + bracket. Out of the wrist
  camera's view. Demo videos and poster re-rendered.
- README architecture diagram reads top to bottom (sensing -> nodes -> controllers -> physics) and is exported to
  docs/media/architecture.svg (plain SVG text) by tools/export_architecture.sh.
- catch_sim.sim_clock.offload_sim_clock: /clock handled by a helper node on an EventsExecutor thread instead of
  each node's MultiThreadedExecutor (108 % -> 7 % of a core per node for /clock alone); monitors spin on an
  EventsExecutor. Idle Python CPU 643 % -> 309 %; run_demo seed 1 complete, color step 5.9 -> 0.4 s.
- tools/node_cpu.py: per-node CPU measurement. Feed-forward table rehashed (torques identical).
- Isaac downgrade checked: not applied (see docs/progress.md).

File: src/catch_description/urdf/scene.urdf.xacro (robot description, xacro)
@@ -126,4 +126,25 @@
     <origin xyz="0 0 -0.014" rpy="${-atan2(-cos(wc_phi), -sin(wc_phi))} 0 0"/>
   </joint>
+  <!-- bracket holding the housing to the gripper base; link frame = Menagerie gripper base frame (the TCP frame is
+       that frame rotated +90 deg about z and raised to the cube centre). Collision boxes 1 mm larger per side. -->
+  <xacro:macro name="bracket_box" params="lo hi grow">
+    <origin xyz="${(lo[0] + hi[0]) / 2} ${(lo[1] + hi[1]) / 2} ${(lo[2] + hi[2]) / 2}"/>
+    <geometry><box size="${hi[0] - lo[0] + 2 * grow} ${hi[1] - lo[1] + 2 * grow} ${hi[2] - lo[2] + 2 * grow}"/></geometry>
+  </xacro:macro>
+  <link name="b_wrist_cam_bracket">
+    <xacro:property name="bk" value="${scene['cameras']['b_wrist_bracket']}"/>
+    <xacro:property name="bk0" value="${bk[0]}"/>
+    <xacro:property name="bk1" value="${bk[1]}"/>
+    <visual><xacro:bracket_box lo="${bk0[0]}" hi="${bk0[1]}" grow="0"/>
+      <material name="b_wrist_bracket_mat"><color rgba="0.32 0.33 0.35 1"/></material></visual>
+    <visual><xacro:bracket_box lo="${bk1[0]}" hi="${bk1[1]}" grow="0"/>
+      <material name="b_wrist_bracket_mat"/></visual>
+    <collision><xacro:bracket_box lo="${bk0[0]}" hi="${bk0[1]}" grow="0.001"/></collision>
+    <collision><xacro:bracket_box lo="${bk1[0]}" hi="${bk1[1]}" grow="0.001"/></collision>
+  </link>
+  <joint name="b_wrist_cam_bracket_joint" type="fixed">
+    <parent link="b_tcp"/><child link="b_wrist_cam_bracket"/>
+    <origin xyz="0 0 ${-(ins['top_z'] + edge / 2)}" rpy="0 0 ${-pi / 2}"/>
+  </joint>
   <xacro:if value="$(arg ros2_control)">
     <ros2_control name="MujocoSystem" type="system">

Commit message: v2.3: B's arm configuration review (planner never changed IK branch: 0 in 310 recorded trials; flips were home <-> ready; elbow-up home-branch ready poses with ik_branch fixed catch 51 % (60 deg) / 56 % (55 deg) vs 100 % for the Phase 1 pose -> Phase 1 stays default, elbow-up poses are reactive.yaml variants; ik_branch free|fixed, CATCH_READY_POSE / CATCH_IK_BRANCH); B waits at home and gets ready at LOAD (prepare_only direct move; demo 9/9, ready 0.5-3.6 s early); wrist depth camera 42x42x23 mm on a clamp mount (optical frame unchanged, camera capsules checked vs MuJoCo and MoveIt meshes); clean RViz default with GT cube markers and B's wrist image (docs/media/rviz.png)

File: src/catch_description/urdf/scene.urdf.xacro (robot description, xacro)
@@ -115,31 +115,39 @@
     <origin xyz="${wc[1]} ${-wc[0]} ${wc_dz}" rpy="${atan2(-cos(wc_phi), -sin(wc_phi))} 0 ${pi / 2}"/>
   </joint>
-  <!-- camera housing (MJCF: visual only, 24 x 30 x 24 mm); collision box 1 mm larger per side for MoveIt -->
+  <!-- wrist camera hardware (scene.yaml b_wrist_camera_parts; MJCF: visual only): camera-frame parts on
+       b_wrist_cam_housing (= the optical frame), mount parts on b_wrist_cam_bracket (= the Menagerie gripper base
+       frame: the TCP frame rotated -90 deg about z and lowered to the base). Collision = each part 1 mm larger per
+       side (MoveIt). Cylinder axis x / y: rotated from z. -->
+  <xacro:macro name="cam_part_geom" params="pt grow">
+    <xacro:property name="sz" value="${pt['size']}"/>
+    <xacro:property name="ax" value="${pt.get('axis', 'z') if pt['type'] == 'cylinder' else 'z'}"/>
+    <origin xyz="${pt['pos'][0]} ${pt['pos'][1]} ${pt['pos'][2]}"
+            rpy="${'0 %r 0' % (pi / 2) if ax == 'x' else ('%r 0 0' % (-pi / 2) if ax == 'y' else '0 0 0')}"/>
+    <geometry>
+      <xacro:if value="${pt['type'] == 'box'}"><box size="${sz[0] + 2 * grow} ${sz[1] + 2 * grow} ${sz[2] + 2 * grow}"/></xacro:if>
+      <xacro:if value="${pt['type'] == 'cylinder'}"><cylinder radius="${sz[0] + grow}" length="${sz[1] + 2 * grow}"/></xacro:if>
+    </geometry>
+  </xacro:macro>
+  <xacro:macro name="cam_parts" params="parts frame">
+    <xacro:if value="${parts}">
+      <xacro:property name="pt" value="${parts[0]}"/>
+      <xacro:if value="${pt['frame'] == frame}">
+        <visual name="wrist_cam_${pt['name']}"><xacro:cam_part_geom pt="${pt}" grow="0"/>
+          <material name="b_wrist_cam_${pt['name']}_mat"><color rgba="${pt['rgba'][0]} ${pt['rgba'][1]} ${pt['rgba'][2]} ${pt['rgba'][3]}"/></material>
+        </visual>
+        <collision name="wrist_cam_${pt['name']}"><xacro:cam_part_geom pt="${pt}" grow="0.001"/></collision>
+      </xacro:if>
+      <xacro:cam_parts parts="${parts[1:]}" frame="${frame}"/>
+    </xacro:if>
+  </xacro:macro>
   <link name="b_wrist_cam_housing">
-    <visual><geometry><box size="0.024 0.030 0.024"/></geometry>
-      <material name="b_wrist_cam_mat"><color rgba="0.1 0.1 0.1 1"/></material></visual>
-    <collision><geometry><box size="0.026 0.032 0.026"/></geometry></collision>
+    <xacro:cam_parts parts="${scene['cameras']['b_wrist_camera_parts']}" frame="camera"/>
   </link>
   <joint name="b_wrist_cam_housing_joint" type="fixed">
     <parent link="b_wrist_cam_optical"/><child link="b_wrist_cam_housing"/>
-    <!-- MJCF housing: 14 mm behind the lens along the view axis, box axes = Menagerie base axes -->
-    <origin xyz="0 0 -0.014" rpy="${-atan2(-cos(wc_phi), -sin(wc_phi))} 0 0"/>
+    <origin xyz="0 0 0" rpy="0 0 0"/>
   </joint>
-  <!-- bracket holding the housing to the gripper base; link frame = Menagerie gripper base frame (the TCP frame is
-       that frame rotated +90 deg about z and raised to the cube centre). Collision boxes 1 mm larger per side. -->
-  <xacro:macro name="bracket_box" params="lo hi grow">
-    <origin xyz="${(lo[0] + hi[0]) / 2} ${(lo[1] + hi[1]) / 2} ${(lo[2] + hi[2]) / 2}"/>
-    <geometry><box size="${hi[0] - lo[0] + 2 * grow} ${hi[1] - lo[1] + 2 * grow} ${hi[2] - lo[2] + 2 * grow}"/></geometry>
-  </xacro:macro>
   <link name="b_wrist_cam_bracket">
-    <xacro:property name="bk" value="${scene['cameras']['b_wrist_bracket']}"/>
-    <xacro:property name="bk0" value="${bk[0]}"/>
-    <xacro:property name="bk1" value="${bk[1]}"/>
-    <visual><xacro:bracket_box lo="${bk0[0]}" hi="${bk0[1]}" grow="0"/>
-      <material name="b_wrist_bracket_mat"><color rgba="0.32 0.33 0.35 1"/></material></visual>
-    <visual><xacro:bracket_box lo="${bk1[0]}" hi="${bk1[1]}" grow="0"/>
-      <material name="b_wrist_bracket_mat"/></visual>
-    <collision><xacro:bracket_box lo="${bk0[0]}" hi="${bk0[1]}" grow="0.001"/></collision>
-    <collision><xacro:bracket_box lo="${bk1[0]}" hi="${bk1[1]}" grow="0.001"/></collision>
+    <xacro:cam_parts parts="${scene['cameras']['b_wrist_camera_parts']}" frame="base"/>
   </link>
   <joint name="b_wrist_cam_bracket_joint" type="fixed">
